Commit message: day 18

File: src/mini_robot_urdf/urdf/mini_robot.urdf (robot description, URDF)
Before this commit: robot mini_robot, 8 links, 7 joints
Joints:
- joint arm_joint: axis 0 1 0 -> 0 0 1

Commit message: day20

File: src/mini_robot_urdf/urdf/mini_robot.urdf (robot description, URDF)
Before this commit: robot mini_robot, 8 links, 7 joints
Joints:
- joint left_wheel_joint: axis (none) -> 0 1 0; type fixed -> continuous
- joint right_wheel_joint: axis (none) -> 0 1 0; type fixed -> continuous

File: src/mini_robot_urdf/xacro/mini_robot.xacro (robot description, xacro)
@@ -7,5 +7,4 @@
   <xacro:property name="wheel_radius" value="0.05" />
   <xacro:property name="wheel_width" value="0.04" />
-  <xacro:property name="wheel_x" value="${base_length / 2 - wheel_radius}" />
   <xacro:property name="wheel_y" value="${base_width / 2 + wheel_width / 2}" />
   <xacro:property name="wheel_z" value="${-base_height / 2}" />
@@ -27,11 +26,7 @@
     </visual>
   </link>
-  <xacro:wheel prefix="front_left" x_pos="${wheel_x}" y_pos="${wheel_y}" z_pos="${wheel_z}"
+  <xacro:wheel prefix="left" x_pos="0" y_pos="${wheel_y}" z_pos="${wheel_z}"
     wheel_radius="${wheel_radius}" wheel_width="${wheel_width}" />
-  <xacro:wheel prefix="front_right" x_pos="${wheel_x}" y_pos="${-wheel_y}" z_pos="${wheel_z}"
-    wheel_radius="${wheel_radius}" wheel_width="${wheel_width}" />
-  <xacro:wheel prefix="rear_left" x_pos="${-wheel_x}" y_pos="${wheel_y}" z_pos="${wheel_z}"
-    wheel_radius="${wheel_radius}" wheel_width="${wheel_width}" />
-  <xacro:wheel prefix="rear_right" x_pos="${-wheel_x}" y_pos="${-wheel_y}" z_pos="${wheel_z}"
+  <xacro:wheel prefix="right" x_pos="0" y_pos="${-wheel_y}" z_pos="${wheel_z}"
     wheel_radius="${wheel_radius}" wheel_width="${wheel_width}" />
 </robot>
