Commit message: day21

File: src/mini_robot_urdf/xacro/mini_robot.xacro (robot description, xacro)
@@ -30,3 +30,21 @@
   <xacro:wheel prefix="right" x_pos="0" y_pos="${-wheel_y}" z_pos="${wheel_z}"
     wheel_radius="${wheel_radius}" wheel_width="${wheel_width}" />
+  <ros2_control
+    name="MiniRobotSystem"
+    type="system">
+    <hardware>
+      <plugin>mock_components/GenericSystem</plugin>
+      <param name="calculate_dynamics">true</param>
+    </hardware>
+    <joint name="left_wheel_joint">
+      <command_interface name="velocity" />
+      <state_interface name="position" />
+      <state_interface name="velocity" />
+    </joint>
+    <joint name="right_wheel_joint">
+      <command_interface name="velocity" />
+      <state_interface name="position" />
+      <state_interface name="velocity" />
+    </joint>
+  </ros2_control>
 </robot>
